Commit message: q management update

File: robot_model/humanoid_mani.urdf (robot description, URDF)
Before this commit: robot humanoid_mani, 8 links, 7 joints
Joints:
- joint rotate_3: origin xyz=-0.02147 -0.0325 -0.025 rpy=0 0 0 -> xyz=-0.02147 -0.0325 -0.025 rpy=1.5708 0 0
- joint rotate_tilt: axis 0.0 -1.0 -0.0 -> 0.0 1.0 -0.0; limit lower=-2.225 upper=0.0 effort=100.0 velocity=1.0 -> lower=0.0 upper=2.225 effort=100.0 velocity=1.0

Commit message: model cfg update

File: robot_model/humanoid_mani.urdf (robot description, URDF)
Before this commit: robot humanoid_mani, 8 links, 7 joints
Links:
- link Head_1: geometry collision mesh filename=file:///home/lwj/colcon_ws/install/humanoid_mani_descriptio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 scale=0.001 0.001 0.001; visual mesh filename=file:///home/lwj/colcon_ws/install/humanoid_mani_descriptio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 scale=0.001 0.001 0.001
- link base_link: geometry collision mesh filename=file:///home/lwj/colcon_ws/install/humanoid_mani_descriptio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 scale=0.001 0.001 0.001; visual mesh filename=file:///home/lwj/colcon_ws/install/humanoid_mani_descriptio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 scale=0.001 0.001 0.001
- link ee_link_1: mass 1.9027076814554607e-07 -> 1.902707681457099e-07; geometry collision mesh filename=file:///home/lwj/colcon_ws/install/humanoid_mani_descriptio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 scale=0.001 0.001 0.001; visual mesh filename=file:///home/lwj/colcon_ws/install/humanoid_mani_descriptio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 scale=0.001 0.001 0.001
- link eye_1: geometry collision mesh filename=file:///home/lwj/colcon_ws/install/humanoid_mani_descriptio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 scale=0.001 0.001 0.001; visual mesh filename=file:///home/lwj/colcon_ws/install/humanoid_mani_descriptio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 scale=0.001 0.001 0.001
- link forearm_1: mass 1.088969578492718 -> 0.7439602672633931; geometry collision mesh filename=file:///home/lwj/colcon_ws/install/humanoid_mani_descriptio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 scale=0.001 0.001 0.001; visual mesh filename=file:///home/lwj/colcon_ws/install/humanoid_mani_descriptio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 scale=0.001 0.001 0.001
- link shoulder_1: geometry collision mesh filename=file:///home/lwj/colcon_ws/install/humanoid_mani_descriptio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 scale=0.001 0.001 0.001; visual mesh filename=file:///home/lwj/colcon_ws/install/humanoid_mani_descriptio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 scale=0.001 0.001 0.001
- link torso_1: geometry collision mesh filename=file:///home/lwj/colcon_ws/install/humanoid_mani_descriptio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 scale=0.001 0.001 0.001; visual mesh filename=file:///home/lwj/colcon_ws/install/humanoid_mani_descriptio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 scale=0.001 0.001 0.001
- link upperarm_1: geometry collision mesh filename=file:///home/lwj/colcon_ws/install/humanoid_mani_descriptio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 scale=0.001 0.001 0.001; visual mesh filename=file:///home/lwj/colcon_ws/install/humanoid_mani_descriptio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 scale=0.001 0.001 0.001
Joints:
- joint ee_dummy: origin xyz=0.0044 -0.144823 -0.020415 rpy=0 0 0 -> xyz=0.004518 -0.164819 -0.020415 rpy=0 0 0
- joint rgb_dummy: origin xyz=0.002 0.017963 0.04 rpy=0 0 0 -> xyz=0.001987 0.017963 0.04 rpy=0 0 0
- joint rotate_1: axis 0.0 -1.0 -0.0 -> 0.000712 -1.0 -0.0; origin xyz=-0.000708 -0.093025 0.10546 rpy=0 0 0 -> xyz=-0.000642 -0.093026 0.10546 rpy=0 0 0
- joint rotate_3: origin xyz=-0.02147 -0.0325 -0.025 rpy=1.5708 0 0 -> xyz=-0.021447 -0.032515 -0.025 rpy=1.5708 0 0
- joint rotate_5: origin xyz=0.02055 -0.1432 0.020499 rpy=0 0 0 -> xyz=0.020652 -0.143185 0.020499 rpy=0 0 0
- joint rotate_tilt: axis 0.0 1.0 -0.0 -> -0.000712 1.0 0.0; origin xyz=0.023041 0.021316 0.14636 rpy=0 0 0 -> xyz=0.023026 0.021333 0.14636 rpy=0 0 0

Commit message: solve urdf linking issue

File: robot_model/humanoid_mani.urdf (robot description, URDF)
Before this commit: robot humanoid_mani, 8 links, 7 joints
Links:
- link Head_1: geometry collision mesh filename=package://humanoid_manipulator/robot_model/meshes/Head_1.stl scale=0.001 0.001 0.001; visual mesh filename=package://humanoid_manipulator/robot_model/meshes/Head_1.stl scale=0.001 0.001 0.001
- link base_link: geometry collision mesh filename=package://humanoid_manipulator/robot_model/meshes/base_link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 scale=0.001 0.001 0.001; visual mesh filename=package://humanoid_manipulator/robot_model/meshes/base_link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 scale=0.001 0.001 0.001
- link ee_link_1: mass 1.902707681457099e-07 -> 1.9027076814554607e-07; geometry collision mesh filename=package://humanoid_manipulator/robot_model/meshes/ee_link_1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 scale=0.001 0.001 0.001; visual mesh filename=package://humanoid_manipulator/robot_model/meshes/ee_link_1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 scale=0.001 0.001 0.001
- link eye_1: geometry collision mesh filename=package://humanoid_manipulator/robot_model/meshes/eye_1.stl scale=0.001 0.001 0.001; visual mesh filename=package://humanoid_manipulator/robot_model/meshes/eye_1.stl scale=0.001 0.001 0.001
- link forearm_1: mass 0.7439602672633931 -> 1.088969578492718; geometry collision mesh filename=package://humanoid_manipulator/robot_model/meshes/forearm_1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 scale=0.001 0.001 0.001; visual mesh filename=package://humanoid_manipulator/robot_model/meshes/forearm_1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 scale=0.001 0.001 0.001
- link shoulder_1: geometry collision mesh filename=package://humanoid_manipulator/robot_model/meshes/shoulder_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 scale=0.001 0.001 0.001; visual mesh filename=package://humanoid_manipulator/robot_model/meshes/shoulder_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 scale=0.001 0.001 0.001
- link torso_1: geometry collision mesh filename=package://humanoid_manipulator/robot_model/meshes/torso_1.s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 scale=0.001 0.001 0.001; visual mesh filename=package://humanoid_manipulator/robot_model/meshes/torso_1.s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 scale=0.001 0.001 0.001
- link upperarm_1: geometry collision mesh filename=package://humanoid_manipulator/robot_model/meshes/upperarm_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 scale=0.001 0.001 0.001; visual mesh filename=package://humanoid_manipulator/robot_model/meshes/upperarm_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 scale=0.001 0.001 0.001
Joints:
- joint ee_dummy: origin xyz=0.004518 -0.164819 -0.020415 rpy=0 0 0 -> xyz=0.0044 -0.144823 -0.020415 rpy=0 0 0
- joint rgb_dummy: origin xyz=0.001987 0.017963 0.04 rpy=0 0 0 -> xyz=0.002 0.017963 0.04 rpy=0 0 0
- joint rotate_1: axis 0.000712 -1.0 -0.0 -> 0.0 -1.0 -0.0; origin xyz=-0.000642 -0.093026 0.10546 rpy=0 0 0 -> xyz=-0.000708 -0.093025 0.10546 rpy=0 0 0
- joint rotate_3: origin xyz=-0.021447 -0.032515 -0.025 rpy=1.5708 0 0 -> xyz=-0.02147 -0.0325 -0.025 rpy=1.5708 0 0
- joint rotate_5: origin xyz=0.020652 -0.143185 0.020499 rpy=0 0 0 -> xyz=0.02055 -0.1432 0.020499 rpy=0 0 0
- joint rotate_tilt: axis -0.000712 1.0 0.0 -> 0.0 1.0 -0.0; origin xyz=0.023026 0.021333 0.14636 rpy=0 0 0 -> xyz=0.023041 0.021316 0.14636 rpy=0 0 0

Commit message: FOR NUC 2

File: robot_model/humanoid_mani.urdf (robot description, URDF)
Before this commit: robot humanoid_mani, 8 links, 7 joints
Joints:
- joint rotate_torso: limit lower=-3.1415 upper=3.1415 effort=100.0 velocity=1.0 -> lower=-1.57 upper=1.57 effort=100.0 velocity=1.0
